File: TLPHnode.sch (KiCad schematic (older format))
At the start: 29 parts, among them P1 Bat, P2 CONN_01X05, SW1 Reset, U1 NCP703, U2 LD39130S, U3 LPS25HB, U4 Si7006-A20, U5 ESP-12E, U6 ISL29035

Commit message: Change Bat to a through-hole connector
  - Add VBat to P2 so that a single connector can
    be used when connecting to a charger/breakout/debug board
  - Use a two-pin through-hole header for VBat to make it
    easy to solder wires rather than use a connector.

On branch AltPower
modified:   TLPHnode-cache.lib
modified:   TLPHnode.kicad_pcb
modified:   TLPHnode.net
modified:   TLPHnode.sch
Parts:
- removed P2: CONN_01X05, rockingdlabs:FPC_conn-5_8x4.9mm_Pitch0.5mm, symbol CONN_01X05
- added P2: CONN_01X06, rockingdlabs:FPC_conn-6_8x4.9mm_Pitch0.5mm, symbol CONN_01X06
- P1: footprint rockingdlabs:JST_PH_S2B-PH-SM4-TB_02x2.00mm_Angled -> Socket_Strips:Socket_Strip_Angled_1x02
Connections:
- net labels added: VBat
- wire segments 102 -> 106
Other:
- moved on the sheet: P1

Commit message: Change battery connection to bare pads
    - Use pin model rather than socket
    - remove 3d model
Parts:
- P1: footprint Socket_Strips:Socket_Strip_Angled_1x02 -> Pin_Headers:Pin_Header_Straight_1x02
Changed lines of the file:
@@
 F 0 "P1" H 1028 2641 50  0000 L CNN
 F 1 "Bat" H 1028 2550 50  0000 L CNN
-F 2 "Socket_Strips:Socket_Strip_Angled_1x02" H 950 2600 50  0001 C CNN
+F 2 "Pin_Headers:Pin_Header_Straight_1x02" H 950 2600 50  0001 C CNN
 F 3 "" H 950 2600 50  0000 C CNN
 	1    950  2600

Commit message: Add Charger control signals to P2
    - All routes removed.

On branch addChrgCtrl
modified:   TLPHnode-cache.lib
modified:   TLPHnode.kicad_pcb
modified:   TLPHnode.net
modified:   TLPHnode.sch
Parts:
- removed P2: CONN_01X06, rockingdlabs:FPC_conn-6_8x4.9mm_Pitch0.5mm, symbol CONN_01X06
- added P2: CONN_01X07, rockingdlabs:FPC_conn-7_8x4.9mm_Pitch0.5mm, symbol CONN_01X07
- R12, R9: value 4.7k -> 10k
Connections:
- net labels added: CHRG, CTRL
- wire segments 106 -> 107
Other:
- moved on the sheet: R12
Changed lines of the file:
@@
 	1    0    0    -1
 $EndComp
-Text Label 3600 6400 0    60   ~ 0
-VCC
-Text Label 3600 6600 0    60   ~ 0
+Text Label 3650 6600 0    60   ~ 0
 GND
-Text Label 3600 6300 0    60   ~ 0
+Text Label 3650 6200 0    60   ~ 0
 RXD
-Text Label 3600 6200 0    60   ~ 0
+Text Label 3650 6100 0    60   ~ 0
 TXD
 Text Label 8300 4300 0    60   ~ 0
@@
 Text Label 8300 4700 0    60   ~ 0
 PGM
-Text Label 3600 6500 0    60   ~ 0
+Text Label 3650 6500 0    60   ~ 0
 PGM
 $Comp
@@
 L R R12
 U 1 1 583BD5E7
-P 7700 3900
-F 0 "R12" H 7770 3946 50  0000 L CNN
-F 1 "4.7k" V 7700 3800 50  0000 L CNN
-F 2 "Resistors_SMD:R_0603" V 7630 3900 50  0001 C CNN
-F 3 "" H 7700 3900 50  0000 C CNN
-	1    7700 3900
+P 8150 5150
+F 0 "R12" H 8220 5196 50  0000 L CNN
+F 1 "10k" V 8150 5050 50  0000 L CNN
+F 2 "Resistors_SMD:R_0603" V 8080 5150 50  0001 C CNN
+F 3 "" H 8150 5150 50  0000 C CNN
+	1    8150 5150
 	1    0    0    -1
 $EndComp
@@
 P 7250 3900
 F 0 "R9" H 7320 3946 50  0000 L CNN
-F 1 "4.7k" V 7250 3800 50  0000 L CNN
+F 1 "10k" V 7250 3800 50  0000 L CNN
 F 2 "Resistors_SMD:R_0603" V 7180 3900 50  0001 C CNN
 F 3 "" H 7250 3900 50  0000 C CNN
@@
 	1    0    0    -1
 $EndComp
-$Comp
-L CONN_01X06 P2
-U 1 1 584F0E69
-P 4000 6450
-F 0 "P2" H 4078 6491 50  0000 L CNN
-F 1 "CONN_01X06" H 4078 6400 50  0000 L CNN
-F 2 "rockingdlabs:FPC_conn-6_8x4.9mm_Pitch0.5mm" H 4000 6450 50  0001 C CNN
-F 3 "" H 4000 6450 50  0000 C CNN
-	1    4000 6450
-	1    0    0    -1
-$EndComp
-Text Label 3600 6700 0    60   ~ 0
+Text Label 3650 6700 0    60   ~ 0
 VBat
 Text Label 1300 2500 0    60   ~ 0
@@
 Connection ~ 2050 3350
 Wire Wire Line
-	3800 6500 3500 6500
-Wire Wire Line
-	3800 6400 3500 6400
-Wire Wire Line
-	3800 6300 3500 6300
-Wire Wire Line
-	3800 6200 3500 6200
-Wire Wire Line
-	3800 6600 3500 6600
+	3850 6500 3550 6500
+Wire Wire Line
+	3850 6200 3550 6200
+Wire Wire Line
+	3850 6100 3550 6100
+Wire Wire Line
+	3850 6600 3550 6600
 Wire Wire Line
 	7200 4300 8500 4300
@@
 	7600 5300 7600 5550
 Wire Wire Line
-	7600 5550 7350 5550
+	7350 5550 8150 5550
 Connection ~ 7350 5550
 Wire Wire Line
@@
 Connection ~ 8050 4700
 Wire Wire Line
-	7200 4600 7700 4600
+	7200 4600 8500 4600
 Wire Wire Line
 	7250 4050 7250 4500
 Wire Wire Line
-	7250 4500 7200 4500
-Wire Wire Line
-	7700 4600 7700 4050
+	7200 4500 8500 4500
 Wire Wire Line
 	7250 3750 7250 3650
@@
 Connection ~ 8050 3650
 Wire Wire Line
-	7700 3750 7700 3650
-Connection ~ 7700 3650
-Wire Wire Line
 	9250 1400 10000 1400
 Connection ~ 9250 1400
@@
 	2300 5700 2300 5800
 Wire Wire Line
-	3800 6700 3500 6700
+	3850 6700 3550 6700
 Connection ~ 1300 2550
 Wire Wire Line
@@
 	1200 2300 1200 2550
 Connection ~ 1200 2550
+$Comp
+L CONN_01X07 P2
+U 1 1 585DBFD0
+P 4050 6400
+F 0 "P2" H 4128 6441 50  0000 L CNN
+F 1 "CONN_01X07" H 4128 6350 50  0000 L CNN
+F 2 "rockingdlabs:FPC_conn-7_8x4.9mm_Pitch0.5mm" H 4050 6400 50  0001 C CNN
+F 3 "" H 4050 6400 50  0000 C CNN
+	1    4050 6400
+	1    0    0    -1
+$EndComp
+Wire Wire Line
+	3850 6300 3550 6300
+Wire Wire Line
+	3850 6400 3550 6400
+Text Label 3650 6300 0    60   ~ 0
+CTRL
+Text Label 3650 6400 0    60   ~ 0
+CHRG
+Connection ~ 7250 4500
+Text Label 8300 4500 0    60   ~ 0
+CHRG
+Wire Wire Line
+	8150 5550 8150 5300
+Connection ~ 7600 5550
+Wire Wire Line
+	8150 5000 8150 4600
+Connection ~ 8150 4600
+Text Label 8300 4600 0    60   ~ 0
+CTRL
 $EndSCHEMATC

Commit message: Checkpoint - Routing complete, 7-pin P2
    - Includes control and monitoring signals for battery charger

On branch addChrgCtrl
modified:   TLPHnode.kicad_pcb
modified:   TLPHnode.net
modified:   TLPHnode.sch
Changed lines of the file:
@@
 Text Label 8300 4700 0    60   ~ 0
 PGM
-Text Label 3650 6500 0    60   ~ 0
+Text Label 3650 6300 0    60   ~ 0
 PGM
 $Comp
@@
 Connection ~ 2050 3350
 Wire Wire Line
-	3850 6500 3550 6500
+	3850 6300 3550 6300
 Wire Wire Line
 	3850 6200 3550 6200
@@
 $EndComp
 Wire Wire Line
-	3850 6300 3550 6300
-Wire Wire Line
 	3850 6400 3550 6400
-Text Label 3650 6300 0    60   ~ 0
+Wire Wire Line
+	3850 6500 3550 6500
+Text Label 3650 6400 0    60   ~ 0
 CTRL
-Text Label 3650 6400 0    60   ~ 0
+Text Label 3600 6500 0    60   ~ 0
 CHRG
 Connection ~ 7250 4500
